File: piezothing.kicad_pcb (KiCad board)
At the start: 2 copper layers, 60 x 20 mm, 11 parts, among them J1 con

Commit message: Added second connector, fixed ring short
Parts:
- added J1: con, Connector_PinHeader_2.54mm:PinHeader_1x02_P2.54mm_Horizontal, B.Cu at (120.8, 72.8)
- moved REF** 128.7 mm to (75.6, 77.6), turned to 180 degrees
- moved G*** 14.1 mm to (123.0, 87.0), turned to 180 degrees
Routing:
- net /A2: track 24.7 -> 44.5 mm
- net /A1: track 59.1 -> 61.8 mm, vias 1 -> 3
- net /K1: track 28.6 -> 29.9 mm
